File: LEDSphere/display_ctrler.kicad_pcb (KiCad board)
At the start: 4 copper layers, 141.9 x 37.1 mm, 46 parts, among them J101 CONN_01x02, J103 Screw_Terminal_01x03, J301 USB_C_Receptacle_USB2.0, J302 Micro_SD_Card, U1 SN74AHC1G14DBVR, U102 W25Q128JVS, U301 USBLC6-2SC6, U303 RP2040, U305 ESP01s, Y301 12MHz

Commit message: display ctrler changes
Parts:
- moved C313 0.43 mm to (183.7, 147.4)
Routing:
- net +3.3V: track 35.2 -> 36.2 mm
- net /VBUS4: track 25.1 -> 25.7 mm
- net GND: track 38.0 -> 38.6 mm
Other:
- board text added: "3.3V"
- board text added: "5V"
- board text added: "Hall"

Commit message: move led terminal up
Parts:
- moved J103 4.65 mm to (210.9, 148.1)
Routing:
- net LED_DATA: track 34.1 -> 29.9 mm
- net +5V: track 44.2 -> 42.9 mm
Changed lines of the file:
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@@
 	(footprint "Footprints:GCT_TAD05-03-1-L-G_REVA"
 		(layer "F.Cu")
-		(at 213.71 151.7975 90)
+		(at 210.87 148.12 90)
 		(property "Reference" "J103"
 			(at -2.725 -4.575 90)
@@
 	)
 	(gr_text "+5V"
-		(at 206.27 156.06 0)
+		(at 214.65 152.27 0)
 		(layer "F.SilkS")
 		(effects
@@
 	)
 	(gr_text "GND"
-		(at 206.52 149 0)
+		(at 214.9 145.21 0)
 		(layer "F.SilkS")
 		(effects
@@
 	)
 	(gr_text "LED"
-		(at 206.76 152.64 0)
+		(at 215.14 148.85 0)
 		(layer "F.SilkS")
 		(effects
@@
 	)
 	(segment
-		(start 212.3535 156.654)
-		(end 213.71 155.2975)
+		(start 188.569474 159.554)
+		(end 191.469474 156.654)
 		(width 0.508)
 		(layer "F.Cu")
@@
 	)
 	(segment
-		(start 172.36 162.14)
-		(end 174.946 159.554)
+		(start 205.836 156.654)
+		(end 210.87 151.62)
 		(width 0.508)
 		(layer "F.Cu")
@@
 	(segment
 		(start 191.469474 156.654)
-		(end 212.3535 156.654)
+		(end 205.836 156.654)
 		(width 0.508)
 		(layer "F.Cu")
@@
 	)
 	(segment
-		(start 188.569474 159.554)
-		(end 191.469474 156.654)
+		(start 172.36 162.14)
+		(end 174.946 159.554)
 		(width 0.508)
 		(layer "F.Cu")
@@
 	)
 	(segment
-		(start 210.265 148.3525)
-		(end 213.71 151.7975)
+		(start 189.532943 148.12)
+		(end 210.87 148.12)
 		(width 0.2)
 		(layer "F.Cu")
@@
 	(segment
 		(start 188.462943 149.19)
-		(end 189.300445 148.3525)
-		(width 0.2)
-		(layer "F.Cu")
-		(net "LED_DATA")
-	)
-	(segment
-		(start 189.300445 148.3525)
-		(end 210.265 148.3525)
+		(end 189.532943 148.12)
 		(width 0.2)
 		(layer "F.Cu")

Commit message: FINAL PUSHES
Parts:
- added D1: LED, LED_SMD:LED_0805_2012Metric, F.Cu at (208.9, 131.2)
- added D2: LED, LED_SMD:LED_0805_2012Metric, F.Cu at (214.6, 131.3)
- added G***: LOGO, LOGO, B.Cu at (88.9, 149.4)
- added R310: 1k, Resistor_SMD:R_0603_1608Metric, F.Cu at (211.2, 131.1)
- added R314: 1k, Resistor_SMD:R_0603_1608Metric, F.Cu at (216.9, 131.2)
- R302, R303: value 5k1 -> 5.1k
Routing:
- net +5V: track 42.9 -> 63.8 mm
- net Net-(D2-K): track 0.00 -> 2.33 mm
- net Net-(D1-K): track 0.00 -> 2.24 mm
- net GND: track 38.6 -> 40.4 mm, vias 35 -> 37
- net +3.3V: track 36.2 -> 37.9 mm, vias 18 -> 19
Other:
- board text added: "Designed by: Ellen Sun"
- board text added: "Eclectronics SP'26 Ellen Sun Jun Park"
- board text added: "LED SPHERE DISPLAY CONTROLLER"

Commit message: update
Parts:
- removed J103: Screw_Terminal_01x03, Footprints:GCT_TAD05-03-1-L-G_REVA
- added J1: Screw_Terminal_01x04, Footprints:PHOENIX_1727036, F.Cu at (214.8, 152.9)
- moved C313 1.70 mm to (184.9, 148.7)
Connections:
- U303 pad 32: LED_DATA -> unconnected-(U303-GPIO21-Pad32)
- U303 pad 34: unconnected-(U303-GPIO22-Pad34) -> LED_CLK
- U303 pad 35: unconnected-(U303-GPIO23-Pad35) -> LED_DATA
Routing:
- net LED_CLK: track 0.00 -> 30.4 mm
- net LED_DATA: track 29.9 -> 31.7 mm
Other:
- board text added: "CLK"
- board text added: "DATA"
- board text removed: "LED"
