File: LEDSphere/display_ctrler.kicad_sch (KiCad schematic)
At the start: 50 parts, among them J101 CONN_01x02, J103 Screw_Terminal_01x03, J301 USB_C_Receptacle_USB2.0, J302 Micro_SD_Card, U1 SN74AHC1G14DBVR, U102 W25Q128JVS, U301 USBLC6-2SC6, U303 RP2040, U305 ESP01s, Y301 12MHz

Commit message: update
Parts:
- removed J103: Screw_Terminal_01x03, Footprints:GCT_TAD05-03-1-L-G_REVA, symbol Connector:Screw_Terminal_01x03
- added J1: Screw_Terminal_01x04, Footprints:PHOENIX_1727036, symbol Connector:Screw_Terminal_01x04
Connections:
- net +5V: now also J1.1 (Pin_1)
- net GND: now also J1.4 (Pin_4)
- net LED_DATA: now also U303.35 (GPIO23), J1.3 (Pin_3); no longer U303.32 (GPIO21)
- net LED_CLK: now reaches U303.34 (GPIO22)
- net LED_CLK: now also J1.2 (Pin_2)
- no-connect marks 27 -> 26
Changed lines of the file:
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@@
 	)
 	(no_connect
+		(at 190.5 124.46)
+	)
+	(no_connect
 		(at 190.5 142.24)
 	)
@@
 	)
 	(no_connect
-		(at 190.5 129.54)
-	)
-	(no_connect
 		(at 190.5 134.62)
 	)
@@
 		(at 139.7 137.16)
 	)
-	(no_connect
-		(at 190.5 127)
-	)
 	(wire
 		(pts
@@
 	(wire
 		(pts
-			(xy 245.11 99.06) (xy 248.92 99.06)
+			(xy 247.65 99.06) (xy 248.92 99.06)
 		)
 		(stroke
@@
 	(wire
 		(pts
-			(xy 245.11 105.41) (xy 245.11 104.14)
-		)
-		(stroke
-			(width 0)
-			(type default)
-		)
-	)
-	(wire
-		(pts
 			(xy 190.5 121.92) (xy 193.04 121.92)
 		)
@@
 	(wire
 		(pts
-			(xy 245.11 104.14) (xy 248.92 104.14)
+			(xy 247.65 106.68) (xy 248.92 106.68)
 		)
 		(stroke
@@
 		)
 	)
-	(global_label "LED_DATA"
-		(shape output)
-		(at 190.5 124.46 0)
+	(global_label "SD_DAT3"
+		(shape bidirectional)
+		(at 76.2 158.75 0)
 		(fields_autoplaced yes)
 		(effects
@@
 		)
 		(property "Intersheetrefs" "${INTERSHEET_REFS}"
-			(at 202.3147 124.46 0)
+			(at 87.4663 158.75 0)
 			(hide yes)
 			(show_name no)
@@
 		)
 	)
-	(global_label "SD_DAT3"
-		(shape bidirectional)
-		(at 76.2 158.75 0)
+	(global_label "I2C0_SDA"
+		(shape output)
+		(at 193.04 101.6 0)
 		(fields_autoplaced yes)
 		(effects
@@
 		)
 		(property "Intersheetrefs" "${INTERSHEET_REFS}"
-			(at 87.4663 158.75 0)
+			(at 204.2005 101.6 0)
 			(hide yes)
 			(show_name no)
@@
 		)
 	)
-	(global_label "I2C0_SDA"
-		(shape output)
-		(at 193.04 101.6 0)
+	(global_label "LED_DATA"
+		(shape input)
+		(at 248.92 104.14 180)
 		(fields_autoplaced yes)
 		(effects
@@
 				(size 1.27 1.27)
 			)
-			(justify left)
+			(justify right)
 		)
 		(property "Intersheetrefs" "${INTERSHEET_REFS}"
-			(at 204.2005 101.6 0)
+			(at 237.1053 104.14 0)
 			(hide yes)
 			(show_name no)
@@
 					(size 1.27 1.27)
 				)
-				(justify left)
+				(justify right)
 			)
 		)
@@
 		)
 	)
-	(global_label "I2C0_SCL"
+	(global_label "LED_CLK"
 		(shape input)
-		(at 231.14 76.2 180)
+		(at 248.92 101.6 180)
 		(fields_autoplaced yes)
 		(effects
@@
 		)
 		(property "Intersheetrefs" "${INTERSHEET_REFS}"
-			(at 220.04 76.2 0)
+			(at 237.952 101.6 0)
 			(hide yes)
 			(show_name no)
@@
 		)
 	)
-	(global_label "LED_DATA"
+	(global_label "I2C0_SCL"
 		(shape input)
-		(at 248.92 101.6 180)
+		(at 231.14 76.2 180)
 		(fields_autoplaced yes)
 		(effects
@@
 		)
 		(property "Intersheetrefs" "${INTERSHEET_REFS}"
-			(at 237.1053 101.6 0)
+			(at 220.04 76.2 0)
 			(hide yes)
 			(show_name no)
@@
 		)
 	)
+	(global_label "LED_CLK"
+		(shape output)
+		(at 190.5 127 0)
+		(fields_autoplaced yes)
+		(effects
+			(font
+				(size 1.27 1.27)
+			)
+			(justify left)
+		)
+		(property "Intersheetrefs" "${INTERSHEET_REFS}"
+			(at 201.468 127 0)
+			(hide yes)
+			(show_name no)
+			(do_not_autoplace no)
+			(effects
+				(font
+					(size 1.27 1.27)
+				)
+				(justify left)
+			)
+		)
+	)
 	(global_label "I2C0_SDA"
 		(shape output)
@@
 		)
 	)
+	(global_label "LED_DATA"
+		(shape output)
+		(at 190.5 129.54 0)
+		(fields_autoplaced yes)
+		(effects
+			(font
+				(size 1.27 1.27)
+			)
+			(justify left)
+		)
+		(property "Intersheetrefs" "${INTERSHEET_REFS}"
+			(at 202.3147 129.54 0)
+			(hide yes)
+			(show_name no)
+			(do_not_autoplace no)
+			(effects
+				(font
+					(size 1.27 1.27)
+				)
+				(justify left)
+			)
+		)
+	)
 	(global_label "SD_DAT0"
 		(shape bidirectional)
@@
 		(lib_name "GND_1")
 		(lib_id "power:GND")
-		(at 245.11 105.41 0)
+		(at 247.65 106.68 0)
 		(unit 1)
 		(body_style 1)
@@
 		(fields_autoplaced yes)
 		(property "Reference" "#PWR0335"
-			(at 245.11 111.76 0)
+			(at 247.65 113.03 0)
 			(hide yes)
 			(show_name no)
@@
 		)
 		(property "Value" "GND"
-			(at 245.11 110.49 0)
+			(at 247.65 111.76 0)
 			(show_name no)
 			(do_not_autoplace no)
@@
 		)
 		(property "Footprint" ""
-			(at 245.11 105.41 0)
+			(at 247.65 106.68 0)
 			(hide yes)
 			(show_name no)
@@
 		)
 		(property "Datasheet" ""
-			(at 245.11 105.41 0)
+			(at 247.65 106.68 0)
 			(hide yes)
 			(show_name no)
@@
 		)
 		(property "Description" "Power symbol creates a global label with name \"GND\" , ground"
-			(at 245.11 105.41 0)
+			(at 247.65 106.68 0)
 			(hide yes)
 			(show_name no)
@@
 	)
 	(symbol
+		(lib_id "Connector:Screw_Terminal_01x04")
+		(at 254 101.6 0)
+		(unit 1)
+		(body_style 1)
+		(exclude_from_sim no)
+		(in_bom yes)
+		(on_board yes)
+		(in_pos_files yes)
+		(dnp no)
+		(fields_autoplaced yes)
+		(property "Reference" "J1"
+			(at 256.54 101.5999 0)
+			(show_name no)
+			(do_not_autoplace no)
+			(effects
+				(font
+					(size 1.27 1.27)
+				)
+				(justify left)
+			)
+		)
+		(property "Value" "Screw_Terminal_01x04"
+			(at 256.54 104.1399 0)
+			(show_name no)
+			(do_not_autoplace no)
+			(effects
+				(font
+					(size 1.27 1.27)
+				)
+				(justify left)
+			)
+		)
+		(property "Footprint" "Footprints:PHOENIX_1727036"
+			(at 254 101.6 0)
+			(hide yes)
+			(show_name no)
+			(do_not_autoplace no)
+			(effects
+				(font
+					(size 1.27 1.27)
+				)
+			)
+		)
+		(property "Datasheet" ""
+			(at 254 101.6 0)
+			(hide yes)
+			(show_name no)
+			(do_not_autoplace no)
+			(effects
+				(font
+					(size 1.27 1.27)
+				)
+			)
+		)
+		(property "Description" "Generic screw terminal, single row, 01x04, script generated (kicad-library-utils/schlib/autogen/connector/)"
+			(at 254 101.6 0)
+			(hide yes)
+			(show_name no)
+			(do_not_autoplace no)
+			(effects
+				(font
+					(size 1.27 1.27)
+				)
+			)
+		)
+		(pin "2"
+		)
+		(pin "4"
+		)
+		(pin "1"
+		)
+		(pin "3"
+		)
+		(instances
+			(project "display_ctrler"
+				(path "/9292a425-4deb-48f6-8b98-43cd7d592040"
+					(reference "J1")
+					(unit 1)
+				)
+			)
+		)
+	)
+	(symbol
 		(lib_id "Device:R")
 		(at 95.25 44.45 180)
@@
 	(symbol
 		(lib_id "power:+5V")
-		(at 245.11 99.06 0)
+		(at 247.65 99.06 0)
 		(unit 1)
 		(body_style 1)
@@
 		(fields_autoplaced yes)
 		(property "Reference" "#PWR02"
-			(at 245.11 102.87 0)
+			(at 247.65 102.87 0)
 			(hide yes)
 			(show_name no)
@@
 		)
 		(property "Value" "+5V"
-			(at 245.11 93.98 0)
+			(at 247.65 93.98 0)
 			(show_name no)
 			(do_not_autoplace no)
@@
 		)
 		(property "Footprint" ""
-			(at 245.11 99.06 0)
+			(at 247.65 99.06 0)
 			(hide yes)
 			(show_name no)
@@
 		)
 		(property "Datasheet" ""
-			(at 245.11 99.06 0)
+			(at 247.65 99.06 0)
 			(hide yes)
 			(show_name no)
@@
 		)
 		(property "Description" "Power symbol creates a global label with name \"+5V\""
-			(at 245.11 99.06 0)
+			(at 247.65 99.06 0)
 			(hide yes)
 			(show_name no)
@@
 					(unit 1)
 				)
-			)
-		)
-	)
-	(symbol
-		(lib_id "Connector:Screw_Terminal_01x03")
-		(at 254 101.6 0)
-		(unit 1)
-		(body_style 1)
-		(exclude_from_sim no)
-		(in_bom yes)
-		(on_board yes)
-		(in_pos_files yes)
-		(dnp no)
-		(fields_autoplaced yes)
-		(property "Reference" "J103"
-			(at 256.54 100.3299 0)
-			(show_name no)
-			(do_not_autoplace no)
-			(effects
-				(font
-					(size 1.27 1.27)
-				)
-				(justify left)
-			)
-		)
-		(property "Value" "Screw_Terminal_01x03"
-			(at 256.54 102.8699 0)
-			(show_name no)
-			(do_not_autoplace no)
-			(effects
-				(font
-					(size 1.27 1.27)
-				)
-				(justify left)
-			)
-		)
-		(property "Footprint" "Footprints:GCT_TAD05-03-1-L-G_REVA"
-			(at 254 101.6 0)
-			(hide yes)
-			(show_name no)
-			(do_not_autoplace no)
-			(effects
-				(font
-					(size 1.27 1.27)
-				)
-			)
-		)
-		(property "Datasheet" "~"
-			(at 254 101.6 0)
-			(hide yes)
-			(show_name no)
-			(do_not_autoplace no)
-			(effects
-				(font
-					(size 1.27 1.27)
-				)
-			)
-		)
-		(property "Description" "Generic screw terminal, single row, 01x03, script generated (kicad-library-utils/schlib/autogen/connector/)"
-			(at 254 101.6 0)
-			(hide yes)
-			(show_name no)
-			(do_not_autoplace no)
-			(effects
-				(font
-					(size 1.27 1.27)
-				)
-			)
-		)
-		(pin "2"
-		)
-		(pin "3"
-		)
-		(pin "1"
-		)
-		(instances
-			(project "display_ctrler"
-				(path "/9292a425-4deb-48f6-8b98-43cd7d592040"
-					(reference "J103")
-					(unit 1)
-				)
