File: power_rx/3_3V_reg.kicad_sch (KiCad schematic)
At the start: 11 parts, among them U102 TPS54202HDDCR

Commit message: buck
Parts:
- C114: value 75pF -> 56pF
- L102: value 33uH -> 10uH
- R112: value 22k -> 22.1k
Changed lines of the file:
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@@
 			)
 		)
-		(property "Value" "22k"
+		(property "Value" "22.1k"
 			(at 217.17 114.3 0)
 			(effects
@@
 			)
 		)
-		(property "Value" "33uH"
+		(property "Value" "10uH"
 			(at 175.26 91.44 90)
 			(effects
@@
 			)
 		)
-		(property "Value" "75pF"
+		(property "Value" "56pF"
 			(at 209.296 106.934 0)
 			(effects
