File: power_rx/power_rx.kicad_sch (KiCad schematic)
At the start: 0 parts

Commit message: start power rx
Parts:
- added C103: 10µF, 50V, Capacitor_SMD:C_1206_3216Metric, symbol Device:C
- added C105, C107, C117: 100nF, Capacitor_SMD:C_0402_1005Metric, symbol Device:C
- added C109: 47pF, Capacitor_SMD:C_0402_1005Metric, symbol Device:C
- added C110: 10pF, Capacitor_SMD:C_0402_1005Metric, symbol Device:C
- added C113, C115: 22µF, 25V, Capacitor_SMD:C_1206_3216Metric, symbol Device:C
- added L103: 33µH, Inductor_SMD:L_Bourns_SRP7028A_7.3x6.6mm, symbol Device:L
- added R101, R105: 100k, Resistor_SMD:R_0402_1005Metric, symbol Device:R
- added R103: 22k, Resistor_SMD:R_0402_1005Metric, symbol Device:R
- added R107: 20k, Resistor_SMD:R_0402_1005Metric, symbol Device:R
- added U101: TPS54202DDC, Package_TO_SOT_SMD:SOT-23-6, symbol Regulator_Switching:TPS54202DDC
- added U105: MH253, my_footprints:MH253, symbol a3144:MH253
- added U106, U111, U112, U113: ~, my_footprints:slot_long, symbol my_symbols:slot1
- added U107, U108, U109, U110: ~, my_footprints:slot_short, symbol my_symbols:slot1
Connections:
- new net +3.3V: C109.1, C110.1, C113.1, C115.1, C117.1, L103.2, R105.2, R107.1, U105.1 (Vcc), U110.1
- new net +5V: U109.1
- new net EN_BC1: R101.2, U101.5 (EN)
- new net FB_BC1: C109.2, C110.2, R103.2, R105.1, U101.4 (FB)
- new net GND: C103.2, C105.2, C113.2, C115.2, C117.2, R103.1, U101.1 (GND), U105.3 (Ground), U106.1, U107.1, U111.1, U112.1, U113.1
- new net Hall: R107.2, U105.2 (Output), U108.1
- new net SW_BC1: C107.2, L103.1, U101.2 (SW)
- new net U_unreg: C103.1, C105.1, R101.1, U101.3 (VIN)
- new net boot_BC1: C107.1, U101.6 (BOOT)
Other:
- added sheet +3.3V Regulator (3_3V_reg.kicad_sch)
- added sheet +5V Regulator (5v_reg.kicad_sch)
- added sheet Receiver Coil (rx_coil.kicad_sch)
- note added: "resistor tolerances 1% or better"

Commit message: buck
Parts:
- removed C103: 10µF, 50V, Capacitor_SMD:C_1206_3216Metric, symbol Device:C
- removed C105, C107: 100nF, Capacitor_SMD:C_0402_1005Metric, symbol Device:C
- removed C109: 47pF, Capacitor_SMD:C_0402_1005Metric, symbol Device:C
- removed C110: 10pF, Capacitor_SMD:C_0402_1005Metric, symbol Device:C
- removed C113, C115: 22µF, 25V, Capacitor_SMD:C_1206_3216Metric, symbol Device:C
- removed L103: 33µH, Inductor_SMD:L_Bourns_SRP7028A_7.3x6.6mm, symbol Device:L
- removed R101, R105: 100k, Resistor_SMD:R_0402_1005Metric, symbol Device:R
- removed R103: 22k, Resistor_SMD:R_0402_1005Metric, symbol Device:R
- removed U101: TPS54202DDC, Package_TO_SOT_SMD:SOT-23-6, symbol Regulator_Switching:TPS54202DDC

Commit message: hall effect sensor
Parts:
- removed C117: 100nF, Capacitor_SMD:C_0402_1005Metric, symbol Device:C
- removed R107: 20k, Resistor_SMD:R_0402_1005Metric, symbol Device:R
- removed U105: MH253, my_footprints:MH253, symbol a3144:MH253
- added C103: 100nF, Capacitor_SMD:C_0402_1005Metric, symbol Device:C
- added R101: 20k, Resistor_SMD:R_0402_1005Metric, symbol Device:R
- added U101: DRV5032FCDBZR, Package_TO_SOT_SMD:SOT-23, symbol Sensor_Magnetic:DRV5033AJxDBZ
Connections:
- net +3.3V: now also C103.1, R101.1, U101.1 (VCC)
- net GND: now also C103.2, U101.3 (GND)
- net Hall: now also R101.2, U101.2 (OUT)
Other:
- moved on the sheet: U108
