File: power_rx/rx_coil.kicad_sch (KiCad schematic)
At the start: 8 parts

Commit message: hall effect sensor
Parts:
- added C201, C202, C203, C204: 100nF, Capacitor_SMD:C_0402_1005Metric, symbol Device:C
- added L201: 6.3uH, symbol Device:L
Connections:
- net coil1: now also L201.2; no longer D101.2 (A), D102.1 (K), U103.1 (pin)
- new net: C201.1, C202.1, C203.1, C204.1, L201.1, U103.1 (pin)
- new net coil2: C201.2, C202.2, C203.2, C204.2, D101.2 (A), D102.1 (K)
Other:
- moved on the sheet: U103, U104
